File: kicad/first.kicad_pcb (KiCad board)
At the start: 2 copper layers, 55.9 x 40.6 mm, 38 parts, among them J1 Conn_01x04_Pin, J10 Conn_01x03_Pin, J11 Conn_01x04_Pin, J2 Conn_01x04_Pin, J3 Conn_01x04_Pin, J4 Conn_01x04_Pin, J5 Conn_01x04_Pin, J6 Conn_01x04_Pin, J7 Conn_01x04_Pin, J8 Conn_01x04_Pin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

Commit message: latest
Parts:
- added drill1: MountingHole_2.1mm, MountingHole:MountingHole_2.1mm, F.Cu at (155.0, 52.5)
- added drill2: MountingHole_2.1mm, MountingHole:MountingHole_2.1mm, F.Cu at (207.0, 52.5)
- added drill3: MountingHole_2.1mm, MountingHole:MountingHole_2.1mm, F.Cu at (155.0, 90.5)
- added drill4: MountingHole_2.1mm, MountingHole:MountingHole_2.1mm, F.Cu at (207.0, 90.5)
- C1, C2, C3: footprint Capacitor_SMD:C_0402_1005Metric -> Capacitor_SMD:C_1206_3216Metric
- D1: footprint LED_SMD:LED_0402_1005Metric -> LED_SMD:LED_1206_3216Metric
- R1, R2, R3, R4, R5, R6, R7, R8: value R_US -> 2.2k; footprint Resistor_SMD:R_0603_1608Metric -> Resistor_SMD:R_1206_3216Metric
- R10, R11, R12, R13, R14, R15, R16, R17, R9: footprint Resistor_SMD:R_0603_1608Metric -> Resistor_SMD:R_1206_3216Metric
- moved J9 24.0 mm to (198.0, 56.9)
- moved C1 22.2 mm to (178.5, 57.8), turned to -90 degrees
- moved Y1 18.2 mm to (184.7, 57.8)
- moved C2 18.2 mm to (191.0, 57.8), turned to -90 degrees
- moved R11 15.5 mm to (181.5, 83.0)
- moved D1 13.2 mm to (187.4, 83.0)
- moved R12 7.51 mm to (203.5, 73.5)
- moved R14 7.51 mm to (203.5, 68.5)
- moved R16 7.51 mm to (203.5, 83.5)
- moved R9 7.51 mm to (203.5, 78.5)
- moved Q1 7.43 mm to (198.9, 78.5)
- moved Q2 7.43 mm to (198.9, 73.5)
- moved Q3 7.43 mm to (198.9, 68.5)
- moved Q4 7.43 mm to (198.9, 83.5)
- moved R10 7.38 mm to (194.5, 78.5)
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Routing:
- net +5V: track 200.0 -> 116.7 mm, vias 6 -> 0
- net Net-(U1-XTAL2/PB7): track 23.1 -> 70.4 mm
- net GND: track 204.3 -> 162.7 mm, vias 2 -> 0
- net /RESET: track 39.6 -> 14.6 mm, vias 1 -> 0
- net +3.3V: track 38.2 -> 56.4 mm, vias 4 -> 0
- net Net-(U1-XTAL1/PB6): track 10.2 -> 26.9 mm, vias 0 -> 2
- net /PD5: track 37.4 -> 21.8 mm
- net /SCK_HV: track 35.2 -> 50.4 mm, vias 1 -> 0
- net /PD6: track 36.4 -> 25.1 mm
- net Net-(U1-PB0): track 23.2 -> 12.6 mm
- net /PD7: track 37.7 -> 28.6 mm
- net /MOSI_HV: track 37.2 -> 42.9 mm
- net /PD0: track 22.5 -> 25.6 mm
- net /MISO_HV: track 30.4 -> 27.5 mm, vias 1 -> 2
- net /PD4: track 25.3 -> 22.5 mm
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Other:
- board size 55.9 x 40.6 mm -> 60.4 x 44.6 mm
- board text added: "3.3V"
- board text added: "5V"
- board text added: "GND"
- board text added: "MISO"
- board text added: "MOSI"
- board text added: "SCK"
- board text added: "SS"
