File: kicad/first.kicad_sch (KiCad schematic)
At the start: 38 parts, among them J1 Conn_01x04_Pin, J10 Conn_01x03_Pin, J11 Conn_01x04_Pin, J2 Conn_01x04_Pin, J3 Conn_01x04_Pin, J4 Conn_01x04_Pin, J5 Conn_01x04_Pin, J6 Conn_01x04_Pin, J7 Conn_01x04_Pin, J8 Conn_01x04_Pin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

Commit message: latest
Parts:
- C1, C2, C3: footprint Capacitor_SMD:C_0402_1005Metric -> Capacitor_SMD:C_1206_3216Metric
- D1: footprint LED_SMD:LED_0402_1005Metric -> LED_SMD:LED_1206_3216Metric
- R1, R2, R3, R4, R5, R6, R7, R8: value R_US -> 2.2k; footprint Resistor_SMD:R_0603_1608Metric -> Resistor_SMD:R_1206_3216Metric
- R10, R11, R12, R13, R14, R15, R16, R17, R9: footprint Resistor_SMD:R_0603_1608Metric -> Resistor_SMD:R_1206_3216Metric
Connections:
- net MISO_LV: now also J11.2 (Pin_2); no longer J11.1 (Pin_1)
- net MOSI_LV: now also J11.3 (Pin_3); no longer J11.2 (Pin_2)
- net SCK_LV: now also J11.1 (Pin_1); no longer J11.3 (Pin_3)
